Commit message: "base_link" is necessary

File: 2r_planar.urdf (robot description, URDF)
Before this commit: robot 2r_planar, 3 links, 2 joints
Links:
- removed link fixed
- added link base_link; visual box size=0.1 0.1 0.1
- link link_1: geometry visual cylinder length=1 radius=0.05
- link link_2: geometry visual cylinder length=1 radius=0.01
Joints:
- joint joint_1: origin xyz=0 0 0.05 rpy=0 0 0 -> xyz=0 0 0.1 rpy=0 0 0; parent fixed -> base_link
- joint joint_2: origin xyz=0 0 0 rpy=0 0 0 -> xyz=0 0 0.1 rpy=0 0 0

Commit message: urdf updated for planar 2r

File: 2r_planar.urdf (robot description, URDF)
Before this commit: robot 2r_planar, 3 links, 2 joints
Links:
- link link_1: geometry visual cylinder length=1 radius=0.01
Joints:
- joint joint_1: axis 0 0 1 -> 1 0 0; origin xyz=0 0 0.1 rpy=0 0 0 -> xyz=0.055 0 0 rpy=0 0 0
- joint joint_2: axis 0 -1 0 -> 1 0 0; origin xyz=0 0 0.1 rpy=0 0 0 -> xyz=-0.02 0 1 rpy=0 0 0
